Commit message: gripper closed postion

File: robotiq_description/urdf/robotiq_2f_85_macro.urdf.xacro (robot description, xacro)
@@ -237,12 +237,11 @@
             <axis xyz="0 -1 0" />
             <origin xyz="0.03060114 0.0 0.05490452" rpy="0 0 0" />
-            <limit lower="0.0" upper="0.8" velocity="0.5" effort="50" />
-        </joint>
-        <joint name="${prefix}robotiq_85_right_knuckle_joint" type="revolute">
+            <limit lower="0.0" upper="${gripper_closed_position}" velocity="0.5" effort="50" />
+        </joint>
+        <joint name="${prefix}robotiq_85_right_knuckle_joint" type="continuous">
             <parent link="${prefix}robotiq_85_base_link" />
             <child link="${prefix}robotiq_85_right_knuckle_link" />
             <axis xyz="0 -1 0" />
             <origin xyz="-0.03060114 0.0 0.05490452" rpy="0 0 0" />
-            <limit lower="-0.8" upper="0.0" velocity="0.5" effort="50" />
             <mimic joint="${prefix}robotiq_85_left_knuckle_joint" multiplier="-1" />
         </joint>
